Commit message: Robot urdf with proper root

File: phippi/urdf/robot.urdf (robot description, URDF)
Before this commit: robot Roboti_algus, 195 links, 194 joints
Joints:
- removed joint 1-1--seib-342
- removed joint 1-1--seib_2-32
- removed joint 1vasak-1--5vasak-12
- removed joint 1vasak-1--seib-92
- removed joint 1vasak-1--seib_2-21
- removed joint 5-1--seib-312
- removed joint 5-1--seib-341
- removed joint Intergy_komplekt-1--Intergy_komplekt-21
- removed joint hammasratas-1--seib_2-51
- removed joint hammasratas-2--seib_2-41
- removed joint hexagonaalne_puks-1--1vasak-11
- removed joint hexagonaalne_puks-1--hexagonaalne_puks-21
- removed joint hexagonaalne_puks-2--1-11
- removed joint kesk plaat-1--2-11
- removed joint kesk plaat-1--3vasak-11
- removed joint kesk plaat-1--seib_2-11
- removed joint kesk plaat-2--roomuk-21
- removed joint kesk plaat-2--seib_2-51
- removed joint panel-3--panel-41
- removed joint pulk-3--panel-11
- removed joint pulk-4--panel-11
- removed joint pulk-4--pulk-21
- removed joint seib-30--mutter-22
- removed joint seib_2-1--seib_2-22
- removed joint seib_2-1--seib_2-41
- removed joint seib_2-2--seib_2-41
- added joint 1-1--seib-341: type fixed, parent 1-11, child seib-341, origin xyz=0.0159999577648 0 0.003 rpy=-2.29637649388 -1.57079632679 0
- added joint 1vasak-1--seib_2-22: type revolute, parent seib_2-23, child 1vasak-12, origin xyz=0.00136168115017 0.00154645791901 0.0016 rpy=3.14159265359 0 -1.55866393809, axis 0 0 -1
- added joint 2-1--pulk-41: type fixed, parent pulk-41, child 2-12, origin xyz=0 0 0.005898 rpy=3.14159265359 0 1.85364910343
- added joint 3-1--pulk-31: type fixed, parent pulk-31, child 3-12, origin xyz=0 0 0.003898 rpy=3.14159265359 0 2.11644671351
- added joint 3-1--seib_2-42: type revolute, parent 3-12, child seib_2-43, origin xyz=0 0 -0.005 rpy=3.14159265359 0 -2.26659028673, axis 0 0 1
- added joint 3vasak-1--pulk-21: type fixed, parent pulk-21, child 3vasak-12, origin xyz=0 0 0.003898 rpy=0 0 -1.29320347691
- added joint 4-1--5-12: type fixed, parent 4-12, child 5-12, origin xyz=0 -0.0537999768328 -0.001 rpy=3.14159265359 0 2.61602157495
- added joint 4-1--seib-312: type revolute, parent 4-12, child seib-312, origin xyz=0 -0.0537999768328 -0.004 rpy=3.02553992101 -1.57079632679 0, axis 0 0 -1
- added joint 4vasak-1--5vasak-12: type fixed, parent 4vasak-12, child 5vasak-12, origin xyz=0 -0.0538000351673 0.001 rpy=3.14159265359 0 2.9947070641
- added joint 5-1--seib-342: type revolute, parent 5-12, child seib-342, origin xyz=0.0662999409233 0 0.004 rpy=2.73207430754 -1.57079632679 0, axis 0 0 1
- added joint 5vasak-1--seib-92: type revolute, parent 5vasak-12, child seib-93, origin xyz=0.0662999594771 0 -0.004 rpy=2.3740236561 1.57079632679 0, axis 0 0 1
- added joint hammasratas-1--1vasak-11: type fixed, parent hammasratas-11, child 1vasak-11, origin xyz=0.003 0 0 rpy=-1.57079632679 -0.368621202939 -1.57079632679
- added joint hammasratas-1--hammasratas-31: type fixed, parent hammasratas-31, child hammasratas-11, origin xyz=0.0596 -0.0300112977917 0.00345133708386 rpy=-1.46864786803 0 -3.14159265359
- added joint hammasratas-2--hammasratas-31: type fixed, parent hammasratas-31, child hammasratas-21, origin xyz=0.0596 0.0300112977917 -0.00345133708386 rpy=2.72014263834 0 3.14159265359
- added joint hammasratas-2--hexagonaalne_puks-11: type prismatic, parent hammasratas-21, child hexagonaalne_puks-11, origin xyz=0.01 -0.00104013312669 -0.00269282607102 rpy=0 0.892220110955 1.57079632679, axis 0 0 -1
- added joint hammasratas-2--seib_2-21: type fixed, parent hammasratas-21, child seib_2-21, origin xyz=0.003 0 0 rpy=1.57079632679 -0.14285347973 1.57079632679
- added joint kesk plaat-1--seib_2-31: type fixed, parent kesk plaat-11, child seib_2-31, origin xyz=0.0641187599584 -0.0512219443348 0.002 rpy=3.14159265359 0 -0.760352338646
- added joint panel-4--panel-21: type fixed, parent panel-21, child panel-41, origin xyz=0.0747513661334 -0.0407237427123 0.045698 rpy=0 0 0.139301424356
- added joint polt-5--mutter-22: type fixed, parent polt-52, child mutter-23, origin xyz=-0.03525 0 0 rpy=-1.57079632679 -1.1777015202 -1.57079632679
- added joint pulk-2--panel-61: type fixed, parent panel-61, child pulk-21, origin xyz=-0.02807905202 -0.0300589875648 -0.138698 rpy=0 0 1.20146759951
- added joint pulk-3--panel-21: type fixed, parent pulk-31, child panel-21, origin xyz=0 0 0 rpy=0 0 2.39489149188
- added joint pulk-3--panel-61: type fixed, parent panel-61, child pulk-31, origin xyz=-0.0641187599584 0.0512219443348 -0.138698 rpy=0 0 -2.39489149188
- added joint pulk-4--pulk-31: type fixed, parent pulk-31, child pulk-41, origin xyz=-0.0517987352503 -0.00456996584113 0 rpy=0 0 -1.90014830697
- added joint seib_2-1--seib_2-31: type fixed, parent seib_2-32, child seib_2-11, origin xyz=-0.0376006439986 0.00787047043389 0 rpy=0 0 0
- added joint seib_2-1--seib_2-33: type fixed, parent seib_2-13, child seib_2-34, origin xyz=0 0 0 rpy=0 0 3.14158409107
- added joint seib_2-1--seib_2-34: type fixed, parent seib_2-35, child seib_2-14, origin xyz=0.0376788170828 -0.0358371358309 0 rpy=0 0 3.14159265359
- joint 1-1--5-12: child 5-12 -> 1-12; origin xyz=0.0159999205826 0 0.0114674 rpy=0 0 -1.17340177208 -> xyz=0.0662999409233 0 -0.001 rpy=0 0 1.17340177208; parent 1-12 -> 5-12
- joint 1-1--polt_2-12: origin xyz=0.0159999205826 0 0.0084674 rpy=1.03714332797 -1.57079632679 0 -> xyz=0 0 -0.003 rpy=1.03714332797 -1.57079632679 0
- joint 1-1--pronks_puks-12: origin xyz=0.00799999914744 -0.0218089045855 0.0114674 rpy=-1.57079632679 0 2.93092354784 -> xyz=-0.00799992143516 -0.0218089295149 0 rpy=-1.57079632679 0 2.93092354784
- joint 1-1--seib-101: origin xyz=0.0159999205826 0 0.0114674 rpy=-1.18982531152 -1.57079632679 0 -> xyz=0 0 0 rpy=-1.18982531152 -1.57079632679 0
- joint 1vasak-1--5vasak-11: origin xyz=0.0160000505952 0 -0.003 rpy=0 0 1.03408566721 -> xyz=0.0160000505952 0 -0.0112 rpy=0 0 1.03408566721
- joint 1vasak-1--polt_2-11: origin xyz=0.0160000505952 0 0 rpy=2.10444932562 1.57079632679 0 -> xyz=0.0160000505952 0 -0.0082 rpy=2.10444932562 1.57079632679 0
- joint 1vasak-1--polt_2-12: origin xyz=0.0159999534186 -0.0028868078445 -0.0171845 rpy=2.47329700633 1.57079632679 0 -> xyz=0.016000013413 0 0 rpy=2.47329700633 1.57079632679 0
- joint 1vasak-1--pronks_puksvasak-11: origin xyz=0.0080000103021 -0.0218089324346 -0.003 rpy=1.57079632679 0 -0.210669105748 -> xyz=0.0080000103021 -0.0218089324346 -0.0112 rpy=1.57079632679 0 -0.210669105748
- joint 1vasak-1--pronks_puksvasak-12: origin xyz=0.00799998029876 -0.0246956474487 -0.0201845 rpy=1.57079632679 0 -0.579515517829 -> xyz=0.00800004029311 -0.0218089017158 -0.003 rpy=1.57079632679 0 -0.579515517829
- joint 1vasak-1--seib-131: origin xyz=0.0160000505952 0 -0.003 rpy=-1.95176734207 1.57079632679 0 -> xyz=0.0160000505952 0 -0.0112 rpy=-1.95176734207 1.57079632679 0
- joint 1vasak-1--seib-61: origin xyz=0.0159999534186 -0.0028868078445 -0.0201845 rpy=-1.18982531152 1.57079632679 0 -> xyz=0.016000013413 0 -0.003 rpy=-1.18982531152 1.57079632679 0
- joint 1vasak-1--seib-91: origin xyz=0.0160000505952 0 -0.003 rpy=1.58292011814 1.57079632679 0 -> xyz=0.0160000505952 0 -0.0112 rpy=1.58292011814 1.57079632679 0
- joint 2-1--polt_2-22: origin xyz=0.0220000057648 0 0.0036 rpy=0.945360719685 -1.57079632679 0 -> xyz=0.0220000057648 0 -0.003 rpy=0.945360719685 -1.57079632679 0
- joint 2-1--pronks_puks-22: origin xyz=0.0110000124717 -0.0262185822848 0.0066 rpy=-1.57079632679 0 1.46055429682 -> xyz=0.0110000124717 -0.0262185822848 0 rpy=-1.57079632679 0 1.46055429682
- joint 2-1--seib-262: origin xyz=0.0220000057648 0 0.0066 rpy=1.46055429682 -1.57079632679 0 -> xyz=0.0220000057648 0 0 rpy=1.46055429682 -1.57079632679 0
- joint 2-1--seib-91: origin xyz=0.0220000057648 0 0.0066 rpy=-1.28794355016 -1.57079632679 0 -> xyz=0.0220000057648 0 0 rpy=-1.28794355016 -1.57079632679 0
- joint 3-1--4-12: origin xyz=-0.0309999737072 0 0.0046 rpy=3.14159265359 0 -2.7757378259 -> xyz=-0.0309999737072 0 -0.002 rpy=3.14159265359 0 -2.7757378259
- joint 3-1--roomuk-21: origin xyz=-0.0444563 0.0724818 -0.0854 rpy=0 0 -0.662513827353 -> xyz=-0.0955173 0.0123441 -0.1669999 rpy=0 0 -0.662513827353
- joint 3-1--seib-282: origin xyz=-0.0309999737072 0 0.0016 rpy=2.65968509332 1.57079632679 0 -> xyz=-0.0309999737072 0 -0.005 rpy=2.65968509332 1.57079632679 0
- joint 3-1--seib-292: origin xyz=-0.0154999889309 -0.0329667749941 0.0046 rpy=2.65968509332 1.57079632679 0 -> xyz=-0.0154999889309 -0.0329667749941 -0.002 rpy=2.65968509332 1.57079632679 0
- joint 3vasak-1--4vasak-12: origin xyz=-0.0310000191072 0 -0.0066 rpy=3.14159265359 0 -1.97616585482 -> xyz=-0.0310000191072 0 0.002 rpy=3.14159265359 0 -1.97616585482
- joint 3vasak-1--seib-32: origin xyz=-0.0310000191072 0 -0.0036 rpy=-1.06171126784 -1.57079632679 0 -> xyz=-0.0310000191072 0 0.005 rpy=-1.06171126784 -1.57079632679 0
- joint 3vasak-1--seib-42: origin xyz=-0.0155003963005 -0.032966976461 -0.0066 rpy=-1.06171126784 -1.57079632679 0 -> xyz=-0.0155003963005 -0.032966976461 0.002 rpy=-1.06171126784 -1.57079632679 0
- joint 3vasak-1--seib_2-32: origin xyz=0 0 -0.0036 rpy=3.14159265359 0 -0.668616461251 -> xyz=0 0 0.005 rpy=3.14159265359 0 -0.668616461251
- joint 4-1--5-11: origin xyz=-1.67507634083e-07 -0.0537998293947 -0.001 rpy=3.14159265359 0 2.45468165407 -> xyz=-1.67507634069e-07 -0.0537998293947 -0.001 rpy=3.14159265359 0 2.45468165407
- joint 4-1--polt-51: origin xyz=-1.67507634083e-07 -0.0537998293947 -0.001 rpy=0.328833748104 1.57079632679 0 -> xyz=-1.67507634069e-07 -0.0537998293947 -0.001 rpy=0.328833748104 1.57079632679 0
- joint 4-1--seib-311: origin xyz=-1.67507634083e-07 -0.0537998293947 -0.004 rpy=-0.328833748104 -1.57079632679 0 -> xyz=-1.67507634097e-07 -0.0537998293947 -0.004 rpy=-0.328833748104 -1.57079632679 0
- joint 4-1--seib-321: origin xyz=-1.67507634083e-07 -0.0537998293947 -0.001 rpy=-0.328833748104 -1.57079632679 0 -> xyz=-1.67507634069e-07 -0.0537998293947 -0.001 rpy=-0.328833748104 -1.57079632679 0
- joint 5-1--pronks_puks-42: origin xyz=-0.03314991622 -0.229726067132 0.005 rpy=-1.57079632679 0 2.73207430754 -> xyz=0.0331500247033 -0.229726097881 0.004 rpy=-1.57079632679 0 2.73207430754
- joint 5-1--seib-302: origin xyz=-0.0662999409233 0 0.008 rpy=2.73207430754 -1.57079632679 0 -> xyz=0 0 0.007 rpy=2.73207430754 -1.57079632679 0
- joint 5-1--seib-332: origin xyz=-0.03314991622 -0.229726067132 0.008 rpy=-2.73207430754 1.57079632679 0 -> xyz=0.0331500247033 -0.229726097881 0.007 rpy=-2.73207430754 1.57079632679 0
- joint 5-1--seib-352: origin xyz=-0.0351999671839 -0.00373992231765 0.008 rpy=2.73207430754 -1.57079632679 0 -> xyz=0.0310999737394 -0.00373995306603 0.007 rpy=2.73207430754 -1.57079632679 0
- joint 5vasak-1--pronks_puksvasak-42: origin xyz=-0.0331503768621 -0.229725994909 -0.005 rpy=1.57079632679 0 -2.3740236561 -> xyz=0.033149582615 -0.229726005569 -0.004 rpy=1.57079632679 0 -2.3740236561
- joint 5vasak-1--seib-102: origin xyz=-0.0351999920408 -0.00373992050436 -0.008 rpy=2.3740236561 1.57079632679 0 -> xyz=0.0310999674363 -0.00373993116412 -0.007 rpy=2.3740236561 1.57079632679 0
- joint 5vasak-1--seib-52: origin xyz=-0.0662999594771 0 -0.008 rpy=2.3740236561 1.57079632679 0 -> xyz=0 0 -0.007 rpy=2.3740236561 1.57079632679 0
- joint 5vasak-1--seib-82: origin xyz=-0.0331503768621 -0.229725994909 -0.008 rpy=-2.3740236561 -1.57079632679 0 -> xyz=0.033149582615 -0.229726005569 -0.007 rpy=-2.3740236561 -1.57079632679 0
- joint Assem2^Roboti_algus-1--camera mount-21: child camera mount-21 -> Assem2^Roboti_algus-11; origin xyz=0 -0.0741699 -0.0315 rpy=3.14159265359 0 3.14159265359 -> xyz=0 -0.0741699 0.056 rpy=3.14159265359 0 3.14159265359; parent Assem2^Roboti_algus-11 -> camera mount-21
- joint Assem2^Roboti_algus-1--camera mount-31: child Assem2^Roboti_algus-11 -> camera mount-31; origin xyz=-0.028 -0.0283589 0.0101288 rpy=0 0 0 -> xyz=0 0.0741699 0.0315 rpy=0 0 0; parent camera mount-31 -> Assem2^Roboti_algus-11
- joint Intergy_komplekt-1--panel-21: child panel-21 -> Intergy_komplekt-11; origin xyz=0.043 -0.0180000006605 0 rpy=1.57079632679 0.120606305828 -1.57079632679 -> xyz=-0.00580613042542 0.0302311967797 0.067698 rpy=-1.69140263262 1.57079632679 0; parent Intergy_komplekt-11 -> panel-21
- joint Intergy_komplekt-2--panel-11: child panel-11 -> Intergy_komplekt-21; origin xyz=-0.0385999 0.0119999637223 0.020784624898 rpy=1.57079632679 -0.752058153458 1.57079632679 -> xyz=-0.032549073044 0.0692442740161 0 rpy=-2.32285448025 -1.57079632679 0; parent Intergy_komplekt-21 -> panel-11
- joint hexagonaalne_puks-1--polt_2-11: origin xyz=0 0.01 0 rpy=2.83067342374 0 -1.57079632679 -> xyz=-0.00144340049579 0.0189845 0.00249995683538 rpy=2.83067342374 0 -1.57079632679
- joint hexagonaalne_puks-1--polt_2-21: origin xyz=0 0.01 0 rpy=0.372782495817 0 1.57079632679 -> xyz=-0.00144340049579 0.0189845 0.00249995683538 rpy=0.372782495817 0 1.57079632679
- joint hexagonaalne_puks-1--seib_4-31: origin xyz=-0.00144332133275 -0.0099995 -0.00250002489196 rpy=2.99896472495 0 -1.57079632679 -> xyz=-0.00288672182854 -0.001015 0 rpy=2.99896472495 0 -1.57079632679
- joint hexagonaalne_puks-2--kesk plaat-21: origin xyz=-0.0122449140064 0.02761615114 -0.013333 rpy=-1.57079632679 0 1.32191870197 -> xyz=-0.0245689282697 0.0531733096138 -0.005133 rpy=-1.57079632679 0 1.32191870197
- joint kesk plaat-1--2vasak-11: origin xyz=0.0239208860696 -0.0300590076949 -0.002 rpy=0 0 2.90706267456 -> xyz=0.088039646028 -0.0812809520298 0 rpy=0 0 2.90706267456
- joint kesk plaat-1--3-11: child 3-12 -> kesk plaat-11; origin xyz=-0.0641187599584 0.0512219443348 -0.002 rpy=3.14159265359 0 -0.278444778376 -> xyz=0 0 -0.0066 rpy=3.14159265359 0 -0.278444778376; parent kesk plaat-11 -> 3-12
- joint kesk plaat-1--hammasratas-31: origin xyz=-0.0123240142634 0.0255571584738 -0.055 rpy=-2.60974520096 -1.57079632679 0 -> xyz=0.051794745695 -0.025664785861 -0.053 rpy=-2.60974520096 -1.57079632679 0
- joint kesk plaat-1--kesk plaat-21: child kesk plaat-11 -> kesk plaat-21; origin xyz=0.0123240142634 -0.0255571584738 -0.0082 rpy=0 0 0 -> xyz=0.0641187599584 -0.0512219443348 0.002 rpy=0 0 0; parent kesk plaat-21 -> kesk plaat-11
- joint kesk plaat-1--seib-21: origin xyz=-0.0123240142634 0.0255571584738 -0.002 rpy=-1.98814550833 1.57079632679 0 -> xyz=0.051794745695 -0.025664785861 0 rpy=-1.98814550833 1.57079632679 0
- joint kesk plaat-1--seib_2-21: origin xyz=0 0 -0.002 rpy=3.14159265359 0 -0.760343741286 -> xyz=0.0641187599584 -0.0512219443348 0 rpy=3.14159265359 0 -0.760343741286
- joint kesk plaat-1--seib_3-101: origin xyz=0.0239208860696 -0.0300590076949 0 rpy=1.98814550833 -1.57079632679 0 -> xyz=0.088039646028 -0.0812809520298 0.002 rpy=1.98814550833 -1.57079632679 0
- joint kesk plaat-1--seib_3-111: origin xyz=-0.02807905202 -0.0300589875648 0 rpy=1.98814550833 -1.57079632679 0 -> xyz=0.0360397079384 -0.0812809318996 0.002 rpy=1.98814550833 -1.57079632679 0
- joint kesk plaat-1--seib_3-121: origin xyz=-0.0641187599584 0.0512219443348 0 rpy=1.98814550833 -1.57079632679 0 -> xyz=0 0 0.002 rpy=1.98814550833 -1.57079632679 0
- joint kesk plaat-1--seib_3-131: origin xyz=-0.029205951208 0.0897588013224 0 rpy=1.98814550833 -1.57079632679 0 -> xyz=0.0349128087504 0.0385368569876 0.002 rpy=1.98814550833 -1.57079632679 0
- joint kesk plaat-2--2-11: origin xyz=0.036244900333 -0.0556161661688 -0.002 rpy=0 0 -2.45882919031 -> xyz=0.0239208860696 -0.0300590076949 0.0062 rpy=0 0 -2.45882919031
- joint kesk plaat-2--2vasak-11: origin xyz=-0.0168819369446 0.0642016428486 0 rpy=3.14159265359 0 -2.49423852766 -> xyz=-0.029205951208 0.0897588013224 0.0082 rpy=3.14159265359 0 -2.49423852766
- joint kesk plaat-2--3vasak-11: origin xyz=-0.051794745695 0.025664785861 0 rpy=3.14159265359 0 0.920204953026 -> xyz=-0.0641187599584 0.0512219443348 0.0082 rpy=3.14159265359 0 0.920204953026
- joint kesk plaat-2--idler_gear-51: origin xyz=-0.0431873211855 0.0367061222934 0 rpy=-0.0588373690606 1.57079632679 0 -> xyz=-0.0555113354489 0.0622632807672 0.0082 rpy=-0.0588373690606 1.57079632679 0
- joint kesk plaat-2--seib-31: origin xyz=0 0 0 rpy=1.98814550833 -1.57079632679 0 -> xyz=-0.0123240142634 0.0255571584738 0.0082 rpy=1.98814550833 -1.57079632679 0
- joint kesk plaat-2--seib_2-21: origin xyz=0.0123240142634 -0.0255571584738 0 rpy=0 0 1.98813694583 -> xyz=0 0 0.0082 rpy=0 0 1.98813694583
- joint kesk plaat-2--seib_2-31: origin xyz=0.0123240142634 -0.0255571584738 0 rpy=3.14159265359 0 2.03663119842 -> xyz=0 0 0.0082 rpy=3.14159265359 0 2.03663119842
- joint kesk plaat-2--seib_2-71: origin xyz=0 0 -0.002 rpy=3.14159265359 0 2.38124031494 -> xyz=-0.0123240142634 0.0255571584738 0.0062 rpy=3.14159265359 0 2.38124031494
- joint kesk plaat-2--seib_2-81: origin xyz=-0.0122449140064 0.02761615114 0 rpy=0 0 1.98814550833 -> xyz=-0.0245689282697 0.0531733096138 0.0082 rpy=0 0 1.98814550833
- joint kesk plaat-2--seib_2-91: origin xyz=0.0122449140064 -0.02761615114 0 rpy=0 0 1.98814550833 -> xyz=-7.91002570179e-05 -0.00205899266617 0.0082 rpy=0 0 1.98814550833
- joint kesk plaat-2--seib_3-141: origin xyz=-0.051794745695 0.025664785861 -0.002 rpy=-1.98814550833 1.57079632679 0 -> xyz=-0.0641187599584 0.0512219443348 0.0062 rpy=-1.98814550833 1.57079632679 0
- joint kesk plaat-2--seib_3-151: origin xyz=-0.0168819369446 0.0642016428486 -0.002 rpy=-1.98814550833 1.57079632679 0 -> xyz=-0.029205951208 0.0897588013224 0.0062 rpy=-1.98814550833 1.57079632679 0
- joint kesk plaat-2--seib_3-81: origin xyz=-0.0157550377566 -0.0556161460386 -0.002 rpy=-1.98814550833 1.57079632679 0 -> xyz=-0.02807905202 -0.0300589875648 0.0062 rpy=-1.98814550833 1.57079632679 0
- joint kesk plaat-2--seib_3-91: origin xyz=0.036244900333 -0.0556161661688 -0.002 rpy=-1.98814550833 1.57079632679 0 -> xyz=0.0239208860696 -0.0300590076949 0.0062 rpy=-1.98814550833 1.57079632679 0
- joint panel-1--panel-31: origin xyz=-0.0373758173397 0.0122088670984 0.002 rpy=0 0 0 -> xyz=-0.0699248903838 0.0814531411145 0.002 rpy=0 0 0
- joint panel-1--panel-61: child panel-61 -> panel-11; origin xyz=0.032549073044 -0.0692442740161 0 rpy=0 0 0 -> xyz=0 0 0.015 rpy=0 0 0; parent panel-11 -> panel-61
- joint panel-6--camera mount-31: child camera mount-31 -> panel-61; origin xyz=0 0 -0.015 rpy=-2.72424347206 -1.57079632679 0 -> xyz=0.028 0.0283589 -0.0101288 rpy=1.57079632679 -1.15344714526 1.57079632679; parent panel-61 -> camera mount-31
- joint roller-1--panel-61: origin xyz=0.0183850240675 -0.0747959267216 -0.013 rpy=0 0 1.98814550833 -> xyz=0.0183850240675 -0.0747959267216 0.002 rpy=0 0 1.98814550833
- joint roller-2--panel-61: origin xyz=0.0504557519309 -0.0460708532388 -0.013 rpy=0 0 1.98814550833 -> xyz=0.0504557519309 -0.0460708532388 0.002 rpy=0 0 1.98814550833
- joint roomuk-2--Intergy_komplekt-21: child Intergy_komplekt-21 -> roomuk-21; origin xyz=0.051061 0.0601377 0.0815999 rpy=1.9721853186 -1.57079632679 0 -> xyz=0.0385999 -0.0119999637223 -0.020784624898 rpy=-1.57079632679 -0.401388991802 -1.57079632679; parent roomuk-21 -> Intergy_komplekt-21
- joint seib-34--spacer-21: origin xyz=-0.001 0 0 rpy=3.14159265359 1.2261870846 1.57079632679 -> xyz=0.004 0 0 rpy=3.14159265359 1.2261870846 1.57079632679
- joint seib_2-1--seib_2-42: child seib_2-43 -> seib_2-13; origin xyz=-0.0938927999998 0.00968360000194 0 rpy=0 0 3.14159265359 -> xyz=0.021077599999 -0.0475366000004 0.0016 rpy=0 0 -3.14159265359; parent seib_2-13 -> seib_2-43
- joint seib_2-3--seib_2-51: child seib_2-31 -> seib_2-51; origin xyz=0.058568 0.0009069 -0.0046 rpy=3.14159265359 0 -2.74849784698 -> xyz=-0.054448289982 -0.0215966851541 -0.0016 rpy=3.14159265359 0 -2.74849784698; parent seib_2-51 -> seib_2-31
- joint seib_2-4--kesk plaat-21: origin xyz=0.0122449140064 -0.02761615114 -0.002 rpy=0 0 1.87501431362 -> xyz=-7.91002570179e-05 -0.00205899266617 0.0062 rpy=0 0 1.87501431362
